File: low_power_gsm-gprs.sch (KiCad schematic (older format))
At the start: 38 parts, among them J1 Conn_Coaxial, J2 SIM_Card, J3 Conn_02x20_Odd_Even, J4 USB_B_Micro, Q1 2N7002, Q2 2N7002, U1 SARA-G450, U2 PL2303SA, U3 LT1764AEQ#PBF

Commit message: Fixed up library name
Parts:
- J2: symbol low_power_gsm-gprs:SIM_Card -> muonpi-kicad-library:SIM_Card
- J3: symbol low_power_gsm-gprs:Conn_02x20_Odd_Even -> muonpi-kicad-library:Conn_02x20_Odd_Even
- J4: symbol Connector:USB_B_Micro -> muonpi-kicad-library:USB_B_Micro
- U1: symbol low_power_gsm-gprs:SARA-G450 -> muonpi-kicad-library:SARA-G450
- U2: symbol low_power_gsm-gprs:PL2303SA -> muonpi-kicad-library:PL2303SA
- U3: symbol low_power_gsm-gprs:LT1764AEQ#PBF -> muonpi-kicad-library:LT1764AEQ#PBF
Changed lines of the file:
@@
 $EndDescr
 $Comp
-L low_power_gsm-gprs:SARA-G450 U1
+L muonpi-kicad-library:SARA-G450 U1
 U 1 1 60B38C8C
 P 2250 1950
@@
 	4250 1000 4450 1000
 $Comp
-L low_power_gsm-gprs:LT1764AEQ#PBF U3
+L muonpi-kicad-library:LT1764AEQ#PBF U3
 U 1 1 60B38314
 P 6550 1400
@@
 	9100 1600 8700 1600
 $Comp
-L low_power_gsm-gprs:PL2303SA U2
+L muonpi-kicad-library:PL2303SA U2
 U 1 1 60B921DF
 P 5500 3900
@@
 	5500 3150 5100 3150
 $Comp
-L Connector:USB_B_Micro J4
+L muonpi-kicad-library:USB_B_Micro J4
 U 1 1 60BD11FB
 P 9400 2750
@@
 Connection ~ 9150 3150
 $Comp
-L low_power_gsm-gprs:SIM_Card J2
+L muonpi-kicad-library:SIM_Card J2
 U 1 1 60B43D6F
 P 4350 5400
@@
 	3650 5950 4400 5950
 $Comp
-L low_power_gsm-gprs:Conn_02x20_Odd_Even J3
+L muonpi-kicad-library:Conn_02x20_Odd_Even J3
 U 1 1 60C7CA54
 P 8850 5050

Commit message: Updated parts library
Parts:
- J4: footprint Connector_USB:USB_Micro-B_Amphenol_10104110_Horizontal -> muonpi-kicad-library:USB_Micro-B_Amphenol_10104110_Horizontal; symbol muonpi-kicad-library:USB_B_Micro -> muonpi-kicad-library:USB_B_Micro_SMD
Changed lines of the file:
@@
 	5500 3150 5100 3150
 $Comp
-L muonpi-kicad-library:USB_B_Micro J4
+L muonpi-kicad-library:USB_B_Micro_SMD J4
 U 1 1 60BD11FB
 P 9400 2750
 F 0 "J4" H 9457 3217 50  0000 C CNN
 F 1 "USB_B_Micro" H 9457 3126 50  0000 C CNN
-F 2 "Connector_USB:USB_Micro-B_Amphenol_10104110_Horizontal" H 9550 2700 50  0001 C CNN
+F 2 "muonpi-kicad-library:USB_Micro-B_Amphenol_10104110_Horizontal" H 9550 2700 50  0001 C CNN
 F 3 "~" H 9550 2700 50  0001 C CNN
 	1    9400 2750

Commit message: Updated footprints to be correct.
Parts:
- J1: footprint Connector_Coaxial:SMA_Amphenol_132289_EdgeMount -> muonpi-kicad-library:SMA_Samtec_SMA-J-P-X-ST-EM1_EdgeMount; symbol Connector:Conn_Coaxial -> muonpi-kicad-library:Conn_Coaxial
- U3: footprint low_power_gsm-gprs:TO-263-5_TabPin3 -> muonpi-kicad-library:DD-PAK-5_L10.6-W10.3-P1.70-LS14.5-BR
Changed lines of the file:
@@
 	1350 1500 1450 1500
 $Comp
-L Connector:Conn_Coaxial J1
+L muonpi-kicad-library:Conn_Coaxial J1
 U 1 1 60BC3720
 P 4650 1000
 F 0 "J1" H 4750 975 50  0000 L CNN
 F 1 "Conn_Coaxial" H 4750 884 50  0000 L CNN
-F 2 "Connector_Coaxial:SMA_Amphenol_132289_EdgeMount" H 4650 1000 50  0001 C CNN
+F 2 "muonpi-kicad-library:SMA_Samtec_SMA-J-P-X-ST-EM1_EdgeMount" H 4650 1000 50  0001 C CNN
 F 3 " ~" H 4650 1000 50  0001 C CNN
 	1    4650 1000
@@
 F 0 "U3" H 6550 1767 50  0000 C CNN
 F 1 "LT1764AEQ#PBF" H 6550 1676 50  0000 C CNN
-F 2 "low_power_gsm-gprs:TO-263-5_TabPin3" H 6550 1750 50  0001 C CNN
+F 2 "muonpi-kicad-library:DD-PAK-5_L10.6-W10.3-P1.70-LS14.5-BR" H 6550 1750 50  0001 C CNN
 F 3 "https://www.mouser.de/datasheet/2/609/1764afb-1268181.pdf" H 6550 1400 50  0001 C CNN
 	1    6550 1400

Commit message: Adjusted Footprints
Parts:
- J2: footprint low_power_gsm-gprs:SIM -> muonpi-kicad-library:SIM
- J3: footprint low_power_gsm-gprs:PinSocket_2x20_P2.54mm_Vertical -> muonpi-kicad-library:PinSocket_2x20_P2.54mm_Vertical
- U1: footprint low_power_gsm-gprs:ublox_SARA-G3_LGA-96 -> muonpi-kicad-library:ublox_SARA-G3_LGA-96
Changed lines of the file:
@@
 F 0 "U1" H 2250 3275 50  0000 C CNN
 F 1 "SARA-G450" H 2250 3184 50  0000 C CNN
-F 2 "low_power_gsm-gprs:ublox_SARA-G3_LGA-96" H 2950 900 50  0001 C CNN
+F 2 "muonpi-kicad-library:ublox_SARA-G3_LGA-96" H 2950 900 50  0001 C CNN
 F 3 "https://www.u-blox.com/sites/default/files/SARA-G450_DataSheet_UBX-18006165.pdf" H 2250 1950 50  0001 C CNN
 	1    2250 1950
@@
 F 0 "J2" H 4980 5500 50  0000 L CNN
 F 1 "SIM_Card" H 4980 5409 50  0000 L CNN
-F 2 "low_power_gsm-gprs:SIM" H 4350 5750 50  0001 C CNN
+F 2 "muonpi-kicad-library:SIM" H 4350 5750 50  0001 C CNN
 F 3 " ~" H 4300 5400 50  0001 C CNN
 	1    4350 5400
@@
 F 0 "J3" H 8900 6167 50  0000 C CNN
 F 1 "Conn_02x20_Odd_Even" H 8900 6076 50  0000 C CNN
-F 2 "low_power_gsm-gprs:PinSocket_2x20_P2.54mm_Vertical" H 8850 5050 50  0001 C CNN
+F 2 "muonpi-kicad-library:PinSocket_2x20_P2.54mm_Vertical" H 8850 5050 50  0001 C CNN
 F 3 "~" H 8850 5050 50  0001 C CNN
 	1    8850 5050

Commit message: Updated footprint reference
Parts:
- U2: footprint Package_SO:SOIC-8_3.9x4.9mm_P1.27mm -> muonpi-kicad-library:SOIC-8_3.9x4.9mm_P1.27mm
Changed lines of the file:
@@
 F 0 "U2" H 5500 4267 50  0000 C CNN
 F 1 "PL2303SA" H 5500 4176 50  0000 C CNN
-F 2 "Package_SO:SOIC-8_3.9x4.9mm_P1.27mm" H 5700 4450 50  0001 C CNN
+F 2 "muonpi-kicad-library:SOIC-8_3.9x4.9mm_P1.27mm" H 5700 4450 50  0001 C CNN
 F 3 "" H 5400 4100 50  0001 C CNN
 	1    5500 3900
